File: Hardware/Mother_Board.brd (EAGLE design)
At the start: 100 x 80 mm, 26 parts, among them IC1 MAX3232CPE, IC2 7805TV, U1 PIC18F26K22-I/SP, U2 25LC1024-E/SM

Commit message: Fixed EEPROM SDI and SDO signals routing.
Connections:
- net N$21: now also U1.16; no longer U1.15
- net N$23: now also U1.15; no longer U1.16
Routing:
- net N$23: track 32.6 -> 37.4 mm
- net N$21: track 24.4 -> 25.5 mm
Changed lines of the file:
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@@
 <signal name="N$21">
 <contactref element="U2" pad="5"/>
-<contactref element="U1" pad="15"/>
-<wire x1="43.8912" y1="13.4112" x2="23.9776" y2="13.4112" width="0.508" layer="1"/>
-<wire x1="46.99" y1="16.51" x2="43.8912" y2="13.4112" width="0.508" layer="1"/>
+<contactref element="U1" pad="16"/>
+<wire x1="41.4528" y1="13.4112" x2="23.9776" y2="13.4112" width="0.508" layer="1"/>
+<wire x1="46.736" y1="18.6944" x2="41.4528" y2="13.4112" width="0.508" layer="1"/>
 <wire x1="23.9776" y1="13.4112" x2="23.9014" y2="13.335" width="0.508" layer="1"/>
+<wire x1="46.736" y1="18.6944" x2="46.99" y2="19.05" width="0.508" layer="1"/>
 </signal>
 <signal name="N$23">
-<contactref element="U1" pad="16"/>
 <contactref element="U2" pad="2"/>
+<contactref element="U1" pad="15"/>
 <wire x1="20.7264" y1="15.8496" x2="17.0688" y2="15.8496" width="0.508" layer="1"/>
 <wire x1="25.1968" y1="20.32" x2="20.7264" y2="15.8496" width="0.508" layer="1"/>
-<wire x1="45.5168" y1="20.32" x2="25.1968" y2="20.32" width="0.508" layer="1"/>
-<wire x1="46.736" y1="19.1008" x2="45.5168" y2="20.32" width="0.508" layer="1"/>
+<wire x1="47.5488" y1="20.32" x2="25.1968" y2="20.32" width="0.508" layer="1"/>
+<wire x1="48.3616" y1="19.5072" x2="47.5488" y2="20.32" width="0.508" layer="1"/>
+<wire x1="48.3616" y1="17.8816" x2="48.3616" y2="19.5072" width="0.508" layer="1"/>
+<wire x1="46.99" y1="16.51" x2="48.3616" y2="17.8816" width="0.508" layer="1"/>
 <wire x1="17.0688" y1="15.8496" x2="16.7386" y2="15.875" width="0.508" layer="1"/>
-<wire x1="46.736" y1="19.1008" x2="46.99" y2="19.05" width="0.508" layer="1"/>
 </signal>
 <signal name="N$24">

Commit message: Routed led to RC0 instead of RE3 (which is input-only pin).
Connections:
- net N$37: now also U1.11; no longer U1.1
Routing:
- net N$37: track 6.62 -> 33.1 mm
Changed lines of the file:
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@@
 <autorouter>
 <pass name="Default">
-<param name="RoutingGrid" value="50mil"/>
+<param name="RoutingGrid" value="6.25mil"/>
 <param name="AutoGrid" value="1"/>
 <param name="Efforts" value="2"/>
 <param name="TopRouterVariant" value="1"/>
 <param name="tpViaShape" value="round"/>
-<param name="PrefDir.1" value="a"/>
+<param name="PrefDir.1" value="*"/>
 <param name="PrefDir.2" value="0"/>
 <param name="PrefDir.3" value="0"/>
@@
 <param name="PrefDir.14" value="0"/>
 <param name="PrefDir.15" value="0"/>
-<param name="PrefDir.16" value="a"/>
+<param name="PrefDir.16" value="-"/>
 <param name="cfVia" value="8"/>
 <param name="cfNonPref" value="5"/>
@@
 <wire x1="21.5392" y1="74.7776" x2="21.59" y2="74.93" width="0.508" layer="1"/>
 </signal>
-<signal name="N$37">
-<contactref element="U1" pad="1"/>
-<contactref element="R5" pad="2"/>
-<wire x1="38.2016" y1="49.5808" x2="39.0144" y2="49.5808" width="0.508" layer="1"/>
-<wire x1="34.544" y1="53.2384" x2="38.2016" y2="49.5808" width="0.508" layer="1"/>
-<wire x1="39.0144" y1="49.5808" x2="39.37" y2="49.53" width="0.508" layer="1"/>
-<wire x1="34.544" y1="53.2384" x2="34.29" y2="53.34" width="0.508" layer="1"/>
-</signal>
-<signal name="N$38">
-<contactref element="JP8" pad="2"/>
-<contactref element="R5" pad="1"/>
-<wire x1="20.32" y1="53.2384" x2="23.9776" y2="53.2384" width="0.508" layer="1"/>
-<wire x1="23.9776" y1="53.2384" x2="24.13" y2="53.34" width="0.508" layer="1"/>
-<wire x1="20.32" y1="53.2384" x2="20.32" y2="53.34" width="0.508" layer="1"/>
-</signal>
 <signal name="N$19">
 <contactref element="U1" pad="9"/>
@@
 <wire x1="6.5024" y1="23.9776" x2="6.35" y2="24.13" width="0.508" layer="16"/>
 </signal>
+<signal name="N$37">
+<contactref element="U1" pad="11"/>
+<contactref element="R5" pad="2"/>
+<wire x1="34.544" y1="34.544" x2="34.544" y2="53.2384" width="0.508" layer="16"/>
+<wire x1="38.608" y1="30.48" x2="34.544" y2="34.544" width="0.508" layer="16"/>
+<wire x1="39.8272" y1="30.48" x2="38.608" y2="30.48" width="0.508" layer="16"/>
+<wire x1="40.64" y1="29.6672" x2="39.8272" y2="30.48" width="0.508" layer="16"/>
+<wire x1="40.64" y1="25.6032" x2="40.64" y2="29.6672" width="0.508" layer="16"/>
+<wire x1="39.4208" y1="24.384" x2="40.64" y2="25.6032" width="0.508" layer="16"/>
+<wire x1="34.544" y1="53.2384" x2="34.29" y2="53.34" width="0.508" layer="16"/>
+<wire x1="39.4208" y1="24.384" x2="39.37" y2="24.13" width="0.508" layer="16"/>
+</signal>
+<signal name="N$38">
+<contactref element="JP8" pad="2"/>
+<contactref element="R5" pad="1"/>
+<wire x1="20.32" y1="53.2384" x2="23.9776" y2="53.2384" width="0.508" layer="1"/>
+<wire x1="23.9776" y1="53.2384" x2="24.13" y2="53.34" width="0.508" layer="1"/>
+<wire x1="20.32" y1="53.2384" x2="20.32" y2="53.34" width="0.508" layer="1"/>
+</signal>
 </signals>
